Commit message: log

File: resource/sample.urdf (robot description, URDF)
Before this commit: robot crobot, 43 links, 42 joints
Joints:
- joint rh_THJ2: parent rh_thhub -> rh_thhu

Commit message: fix urdf demo

File: resource/sample.urdf (robot description, URDF)
Before this commit: robot crobot, 43 links, 42 joints
Joints:
- joint rh_THJ2: parent rh_thhu -> rh_thhub

Commit message: forward kinematics

File: resource/sample.urdf (robot description, URDF)
Before this commit: robot crobot, 43 links, 42 joints
Links:
- link base_link: geometry collision mesh filename=./resource/mesh/universal/base.stl; visual mesh filename=./resource/mesh/universal/base.stl
- link forearm_link: geometry collision mesh filename=./resource/mesh/universal/forearm.stl; visual mesh filename=./resource/mesh/universal/forearm.stl
- link rh_ffdistal: geometry collision mesh filename=./resource/mesh/shadow/F1.stl scale=0.001 0.001 0.001; visual mesh filename=./resource/mesh/shadow/F1.stl scale=0.001 0.001 0.001
- link rh_ffknuckle: geometry collision cylinder length=0.014 radius=0.007; visual mesh filename=./resource/mesh/shadow/knuckle.stl scale=0.001 0.001 0.001
- link rh_ffmiddle: geometry collision cylinder length=0.025 radius=0.007; collision sphere radius=0.007
- link rh_ffproximal: geometry collision cylinder length=0.040 radius=0.007; visual mesh filename=./resource/mesh/shadow/F3.stl scale=0.001 0.001 0.001
- link rh_forearm: geometry collision box size=0.07 0.07 0.07; collision cylinder length=0.184 radius=0.07
- link rh_lfdistal: geometry collision mesh filename=./resource/mesh/shadow/F1.stl scale=0.001 0.001 0.001; visual mesh filename=./resource/mesh/shadow/F1.stl scale=0.001 0.001 0.001
- link rh_lfknuckle: geometry collision cylinder length=0.014 radius=0.007; visual mesh filename=./resource/mesh/shadow/knuckle.stl scale=0.001 0.001 0.001
- link rh_lfmetacarpal: geometry collision box size=0.018 0.024 0.040; visual mesh filename=./resource/mesh/shadow/lfmetacarpal.stl scale=0.001 0.001 0.001
- link rh_lfmiddle: geometry collision cylinder length=0.025 radius=0.007; collision sphere radius=0.007
- link rh_lfproximal: geometry collision cylinder length=0.040 radius=0.007; visual mesh filename=./resource/mesh/shadow/F3.stl scale=0.001 0.001 0.001
- link rh_mfdistal: geometry collision mesh filename=./resource/mesh/shadow/F1.stl scale=0.001 0.001 0.001; visual mesh filename=./resource/mesh/shadow/F1.stl scale=0.001 0.001 0.001
- link rh_mfknuckle: geometry collision cylinder length=0.014 radius=0.007; visual mesh filename=./resource/mesh/shadow/knuckle.stl scale=0.001 0.001 0.001
- link rh_mfmiddle: geometry collision cylinder length=0.025 radius=0.007; collision sphere radius=0.007
- link rh_mfproximal: geometry collision cylinder length=0.040 radius=0.007; visual mesh filename=./resource/mesh/shadow/F3.stl scale=0.001 0.001 0.001
- link rh_palm: geometry collision box size=0.018 0.024 0.004; collision box size=0.020 0.024 0.040
- link rh_rfdistal: geometry collision mesh filename=./resource/mesh/shadow/F1.stl scale=0.001 0.001 0.001; visual mesh filename=./resource/mesh/shadow/F1.stl scale=0.001 0.001 0.001
- link rh_rfknuckle: geometry collision cylinder length=0.014 radius=0.007; visual mesh filename=./resource/mesh/shadow/knuckle.stl scale=0.001 0.001 0.001
- link rh_rfmiddle: geometry collision cylinder length=0.025 radius=0.007; collision sphere radius=0.007
- link rh_rfproximal: geometry collision cylinder length=0.040 radius=0.007; visual mesh filename=./resource/mesh/shadow/F3.stl scale=0.001 0.001 0.001
- link rh_thdistal: geometry collision mesh filename=./resource/mesh/shadow/TH1_z.stl scale=0.001 0.001 0.001; visual mesh filename=./resource/mesh/shadow/TH1_z.stl scale=0.001 0.001 0.001
- link rh_thmiddle: geometry collision cylinder length=0.018 radius=0.011; collision sphere radius=0.011
- link rh_thproximal: geometry collision cylinder length=0.018 radius=0.012; visual mesh filename=./resource/mesh/shadow/TH3_z.stl scale=0.001 0.001 0.001
- link rh_wrist: geometry collision box size=0.027 0.018 0.010; collision box size=0.027 0.018 0.010
- link shoulder_link: geometry collision mesh filename=./resource/mesh/universal/shoulder.stl; visual mesh filename=./resource/mesh/universal/shoulder.stl
- link upper_arm_link: geometry collision mesh filename=./resource/mesh/universal/upperarm.stl; visual mesh filename=./resource/mesh/universal/upperarm.stl
- link wrist_1_link: geometry collision mesh filename=./resource/mesh/universal/wrist1.stl; visual mesh filename=./resource/mesh/universal/wrist1.stl
- link wrist_2_link: geometry collision mesh filename=./resource/mesh/universal/wrist2.stl; visual mesh filename=./resource/mesh/universal/wrist2.stl
- link wrist_3_link: geometry collision mesh filename=./resource/mesh/universal/wrist3.stl; visual mesh filename=./resource/mesh/universal/wrist3.stl
